File: lulu-1_pcb/lulu-1_datalogger_pcb/lulu-1_datalogger_pcb.kicad_pcb (KiCad board)
At the start: 2 copper layers, 44 x 84 mm, 40 parts, among them J1 SD_Card_Receptacle, J3 USB_C_Receptacle_USB2.0_16P, J4 Conn_01x20_Socket, J5 Screw_Terminal, SW1 SW_Nidec_CAS-120A1, U1 STM32F401RETx, U2 BMP280, U3 MPU-6050, U4 W25Q16JVSS, U5 LP3982ILD-3.3, Y1 25 Mhz, Y2 32 Khz

Commit message: Replaced footprint and symbol for USB with part that i am ordering
Parts:
- removed C1, C2, C3, C4: 100 nF, Capacitor_SMD:C_0805_2012Metric
- removed C10, C17, C19: 2.2uF, Capacitor_SMD:C_0805_2012Metric
- removed C11, C12: 100nf, Capacitor_SMD:C_0805_2012Metric
- removed C13, C5: 10nF, Capacitor_SMD:C_0805_2012Metric
- removed C14, C15: 0.1uF, Capacitor_SMD:C_0805_2012Metric
- removed C16: 2.2nF, Capacitor_SMD:C_0805_2012Metric
- removed C18: 33nF, Capacitor_SMD:C_0805_2012Metric
- removed C6, C7: 20pF, Capacitor_SMD:C_0805_2012Metric
- removed C8, C9: 1.5pF, Capacitor_SMD:C_0805_2012Metric
- removed J1: SD_Card_Receptacle, Connector_Card:SD-SIM_microSD-microSIM_Molex_104168-1620
- removed J3: USB_C_Receptacle_USB2.0_16P, Connector_USB:USB_C_Receptacle_Amphenol_12401548E4-2A
- removed J4: Conn_01x20_Socket, Connector:FanPinHeader_1x04_P2.54mm_Vertical
- removed J5: Screw_Terminal, TerminalBlock:TerminalBlock_Altech_AK300-3_P5.00mm
- removed R1, R6, R7, R8: 10K, Resistor_SMD:R_0805_2012Metric
- removed R2, R5: 10k, Resistor_SMD:R_0805_2012Metric
- removed R3, R4: 5.1k, Resistor_SMD:R_0805_2012Metric
- removed R9: 100k, Resistor_SMD:R_0805_2012Metric
- removed SW1: SW_Nidec_CAS-120A1, Button_Switch_SMD:Nidec_Copal_CAS-120A
- removed U1: STM32F401RETx, Package_QFP:LQFP-64_10x10mm_P0.5mm
- removed U2: BMP280, Package_LGA:Bosch_LGA-8_2x2.5mm_P0.65mm_ClockwisePinNumbering
- removed U3: MPU-6050, Sensor_Motion:InvenSense_QFN-24_4x4mm_P0.5mm
- removed U4: W25Q16JVSS, Package_SO:SOIC-8_5.23x5.23mm_P1.27mm
- removed U5: LP3982ILD-3.3, Package_SON:WSON-8-1EP_3x2.5mm_P0.5mm_EP1.2x1.5mm_PullBack_ThermalVias
- removed Y1: 25 Mhz, Crystal:Crystal_AT310_D3.0mm_L10.0mm_Horizontal
- removed Y2: 32 Khz, Crystal:Crystal_AT310_D3.0mm_L10.0mm_Horizontal
Other:
- board outline removed

Commit message: removed usb bus pins from mcu
Parts:
- added C1: 20pF, Capacitor_SMD:C_0805_2012Metric, F.Cu at (175.7, 64.0)
- added C10: 10nF, Capacitor_SMD:C_0805_2012Metric, F.Cu at (180.1, 70.0)
- added C11: 2.2uF, Capacitor_SMD:C_0805_2012Metric, F.Cu at (180.1, 73.0)
- added C12: 33nF, Capacitor_SMD:C_0805_2012Metric, F.Cu at (180.1, 76.0)
- added C13: 2.2uF, Capacitor_SMD:C_0805_2012Metric, F.Cu at (180.1, 79.0)
- added C14: 10nF, Capacitor_SMD:C_0805_2012Metric, F.Cu at (180.1, 82.0)
- added C15: 100nf, Capacitor_SMD:C_0805_2012Metric, F.Cu at (184.6, 64.0)
- added C16: 0.1uF, Capacitor_SMD:C_0805_2012Metric, F.Cu at (184.6, 67.0)
- added C17: 100nf, Capacitor_SMD:C_0805_2012Metric, F.Cu at (184.6, 70.0)
- added C18: 2.2nF, Capacitor_SMD:C_0805_2012Metric, F.Cu at (184.6, 73.0)
- added C19: 0.1uF, Capacitor_SMD:C_0805_2012Metric, F.Cu at (184.6, 76.0)
- added C2: 20pF, Capacitor_SMD:C_0805_2012Metric, F.Cu at (175.7, 67.0)
- added C3: 1.5pF, Capacitor_SMD:C_0805_2012Metric, F.Cu at (175.7, 70.0)
- added C4: 1.5pF, Capacitor_SMD:C_0805_2012Metric, F.Cu at (175.7, 73.0)
- added C5: 100 nF, Capacitor_SMD:C_0805_2012Metric, F.Cu at (175.7, 76.0)
- added C6: 2.2uF, Capacitor_SMD:C_0805_2012Metric, F.Cu at (175.7, 79.0)
- added C7: 100 nF, Capacitor_SMD:C_0805_2012Metric, F.Cu at (175.7, 82.0)
- added C8: 100 nF, Capacitor_SMD:C_0805_2012Metric, F.Cu at (180.1, 64.0)
- added C9: 100 nF, Capacitor_SMD:C_0805_2012Metric, F.Cu at (180.1, 67.0)
- added J1: B2B-XH-A, B2B_XH_A:JST_B2B-XH-A, F.Cu at (202.3, 56.9)
- added J2: SBH11-PBPC-D10-ST-BK, SBH11_PBPC_D10_ST_BK:SULLINS_SBH11-PBPC-D10-ST-BK, F.Cu at (224.8, 58.6)
- added J3: MEM2067-02-180-00-A_REVB, MEM2067_02_180_00_A:GCT_MEM2067-02-180-00-A_REVB, F.Cu at (227.5, 91.5)
- added R1: 10k, Resistor_SMD:R_0805_2012Metric, F.Cu at (189.0, 63.9)
- added R2: 10K, Resistor_SMD:R_0805_2012Metric, F.Cu at (189.0, 66.9)
- added R3: 10k, Resistor_SMD:R_0805_2012Metric, F.Cu at (189.0, 69.8)
- added R4: 10K, Resistor_SMD:R_0805_2012Metric, F.Cu at (189.0, 72.8)
- added R5: 10K, Resistor_SMD:R_0805_2012Metric, F.Cu at (189.0, 75.7)
- added R6: 10K, Resistor_SMD:R_0805_2012Metric, F.Cu at (189.0, 78.7)
- added R7: 100k, Resistor_SMD:R_0805_2012Metric, F.Cu at (189.0, 81.6)
- added SW1: SW_Nidec_CAS-120A1, Button_Switch_SMD:Nidec_Copal_CAS-120A, F.Cu at (244.5, 58.5)
- added U1: STM32F401RETx, Package_QFP:LQFP-64_10x10mm_P0.5mm, F.Cu at (226.5, 73.0)
- added U2: BAT54LT1G, footprints:SOT-23-3_1P4X3P040_ONS, F.Cu at (199.4, 63.4)
- added U3: LP3982ILD-3.3, Package_SON:WSON-8-1EP_3x2.5mm_P0.5mm_EP1.2x1.5mm_PullBack_ThermalVias, F.Cu at (204.2, 63.9)
- added U4: BMP280, Package_LGA:Bosch_LGA-8_2x2.5mm_P0.65mm_ClockwisePinNumbering, F.Cu at (239.0, 68.5)
- added U5: MPU-6050, Sensor_Motion:InvenSense_QFN-24_4x4mm_P0.5mm, F.Cu at (238.8, 77.0)
- added U6: W25Q16JVSS, Package_SO:SOIC-8_5.23x5.23mm_P1.27mm, F.Cu at (208.0, 87.0)
- added Y1: 25 Mhz, Crystal:Crystal_AT310_D3.0mm_L10.0mm_Horizontal, F.Cu at (212.2, 76.5)
- added Y2: 32 Khz, Crystal:Crystal_AT310_D3.0mm_L10.0mm_Horizontal, F.Cu at (212.2, 70.7)
